File: EVmulator_T85_Proto.brd (EAGLE design)
At the start: 22 x 26 mm, 24 parts, among them Q2 DMN3404L-7, U1 ATTINY85V

Commit message: Finished compact version
Parts:
- added J2: (no value), Eigene-Rietig:TAG-CONNECT_TC2030-MCP-NL
Connections:
- new net !RESET: J2.5
- new net MISO: J2.1
- new net MOSI: J2.4
- new net SCK: J2.3
- new net VCC: J2.2
- net GND: now also J2.6
Changed lines of the file:
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@@
 <attribute name="VALUE" x="12.5" y="27.5" size="0.6096" layer="27" font="vector" ratio="20" rot="R90" align="top-center"/>
+</element>
+<element name="J2" library="Eigene-Rietig" library_urn="urn:adsk.eagle:library:40964436" package="TAG-CONNECT_TC2030-MCP-NL" package3d_urn="urn:adsk.eagle:package:41146494/1" value="" x="1" y="-8.5" smashed="yes">
+<attribute name="NAME" x="0.365" y="-7.23" size="1.27" layer="25"/>
 </element>
 </elements>
@@
 <via x="12.5" y="21.5" extent="1-16" drill="0.3"/>
 <contactref element="Q2" pad="2"/>
+<contactref element="J2" pad="6"/>
+<wire x1="15" y1="21.5" x2="21" y2="25" width="0" layer="19" extent="1-1"/>
+<wire x1="12.5" y1="21.5" x2="15" y2="21.5" width="0" layer="19" extent="1-1"/>
+<wire x1="11.5" y1="22.05" x2="12.5" y2="21.5" width="0" layer="19" extent="1-1"/>
+<wire x1="11" y1="21" x2="11.5" y2="22.05" width="0" layer="19" extent="1-1"/>
+<wire x1="11.5" y1="20" x2="11" y2="21" width="0" layer="19" extent="1-1"/>
+<wire x1="9" y1="20" x2="11" y2="21" width="0" layer="19" extent="1-1"/>
+<wire x1="15.5" y1="18" x2="15" y2="21.5" width="0" layer="19" extent="1-1"/>
+<wire x1="16.65" y1="18" x2="15.5" y2="18" width="0" layer="19" extent="1-1"/>
+<wire x1="16.5" y1="14" x2="16.65" y2="18" width="0" layer="19" extent="1-1"/>
+<wire x1="18.5" y1="12.5" x2="16.5" y2="14" width="0" layer="19" extent="1-1"/>
+<wire x1="16" y1="11" x2="17.865" y2="11.81" width="0" layer="19" extent="1-1"/>
+<wire x1="13.5" y1="11" x2="16" y2="11" width="0" layer="19" extent="1-1"/>
+<wire x1="11.5" y1="10.5" x2="13.5" y2="11" width="0" layer="19" extent="1-1"/>
+<wire x1="10.65" y1="9.5" x2="11.5" y2="10.5" width="0" layer="19" extent="1-1"/>
+<wire x1="11.5" y1="8.5" x2="10.65" y2="9.5" width="0" layer="19" extent="1-1"/>
+<wire x1="10.65" y1="7.5" x2="11.5" y2="8.5" width="0" layer="19" extent="1-1"/>
+<wire x1="10" y1="6" x2="10.65" y2="7.5" width="0" layer="19" extent="1-1"/>
+<wire x1="10.5" y1="5" x2="10" y2="6" width="0" layer="19" extent="1-1"/>
+<wire x1="11.5" y1="6" x2="10.5" y2="5" width="0" layer="19" extent="1-1"/>
+<wire x1="11.5" y1="4" x2="10.5" y2="5" width="0" layer="19" extent="1-1"/>
+<wire x1="9" y1="5" x2="10" y2="6" width="0" layer="19" extent="1-1"/>
+<wire x1="7.85" y1="5" x2="9" y2="5" width="0" layer="19" extent="1-1"/>
+<wire x1="10.5" y1="12.5" x2="11.5" y2="10.5" width="0" layer="19" extent="1-1"/>
+<wire x1="8.346" y1="12.105" x2="10.5" y2="12.5" width="0" layer="19" extent="1-1"/>
+<wire x1="6.5" y1="12" x2="8.346" y2="12.105" width="0" layer="19" extent="1-1"/>
+<wire x1="3" y1="11" x2="6.5" y2="12" width="0" layer="19" extent="1-1"/>
+<wire x1="8.5" y1="25" x2="11.5" y2="22.05" width="0" layer="19" extent="1-1"/>
+<wire x1="6.5" y1="23.95" x2="8.5" y2="25" width="0" layer="19" extent="1-1"/>
+<wire x1="5" y1="24.5" x2="6.5" y2="23.95" width="0" layer="19" extent="1-1"/>
+<wire x1="3.5" y1="23.95" x2="5" y2="24.5" width="0" layer="19" extent="1-1"/>
+<wire x1="1" y1="25" x2="3.5" y2="23.95" width="0" layer="19" extent="1-1"/>
+<wire x1="16" y1="1.5" x2="11.5" y2="4" width="0" layer="19" extent="1-1"/>
+<wire x1="17.5" y1="1.65" x2="16" y2="1.5" width="0" layer="19" extent="1-1"/>
+<wire x1="19.5" y1="1.65" x2="17.5" y2="1.65" width="0" layer="19" extent="1-1"/>
+<wire x1="21" y1="1.5" x2="19.5" y2="1.65" width="0" layer="19" extent="1-1"/>
+<wire x1="1" y1="1" x2="7.85" y2="5" width="0" layer="19" extent="1-1"/>
+<wire x1="4.81" y1="-7.865" x2="1" y2="1" width="0" layer="19" extent="1-1"/>
 </signal>
 <signal name="N$1">
@@
 <wire x1="9.6" y1="23.95" x2="11.5" y2="23.95" width="0.3" layer="1"/>
 </signal>
+<signal name="MOSI">
+<contactref element="J2" pad="4"/>
+</signal>
+<signal name="!RESET">
+<contactref element="J2" pad="5"/>
+</signal>
+<signal name="SCK">
+<contactref element="J2" pad="3"/>
+</signal>
+<signal name="VCC">
+<contactref element="J2" pad="2"/>
+</signal>
+<signal name="MISO">
+<contactref element="J2" pad="1"/>
+</signal>
 </signals>

Commit message: changed silkscreen for the 3pin header on both boards. Updated gerbers.
Parts:
- removed J2: (no value), Eigene-Rietig:TAG-CONNECT_TC2030-MCP-NL
- Q2: value DMN3404L-7 -> 5.8A/30V/35mΩ
- U1: device Eigene-Rietig:SOIC8 -> Eigene-Rietig:SOIC8_200
Connections:
- removed net !RESET: J2.5
- removed net MISO: J2.1
- removed net MOSI: J2.4
- removed net SCK: J2.3
- removed net VCC: J2.2
- net GND: no longer J2.6
Changed lines of the file:
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@@
 <layer number="156" name="DXF0409-TOP" color="7" fill="1" visible="no" active="no"/>
 <layer number="157" name="DXF0409-BOTTOM" color="7" fill="1" visible="no" active="no"/>
+<layer number="158" name="FaceMMeas" color="3" fill="1" visible="no" active="no"/>
+<layer number="159" name="Geh-Bear2" color="1" fill="7" visible="no" active="no"/>
+<layer number="160" name="Topologie" color="9" fill="1" visible="no" active="no"/>
+<layer number="161" name="tomplace2" color="7" fill="1" visible="no" active="no"/>
 <layer number="166" name="AntennaArea" color="7" fill="1" visible="no" active="yes"/>
 <layer number="168" name="4mmHeightArea" color="7" fill="1" visible="no" active="yes"/>
@@
 <layer number="250" name="Descript" color="3" fill="1" visible="no" active="no"/>
 <layer number="251" name="SMDround" color="12" fill="11" visible="no" active="no"/>
+<layer number="252" name="BR-BS" color="7" fill="1" visible="no" active="no"/>
+<layer number="253" name="Extra" color="7" fill="1" visible="no" active="no"/>
 <layer number="254" name="cooling" color="7" fill="1" visible="no" active="yes"/>
 <layer number="255" name="routoute" color="7" fill="1" visible="no" active="yes"/>
@@
 <attribute name="VALUE" x="5.6001" y="19.5" size="0.02" layer="27" rot="R180"/>
 </element>
-<element name="U1" library="Eigene-Rietig" library_urn="urn:adsk.eagle:library:40964436" package="SOIC8" package3d_urn="urn:adsk.eagle:package:41055619/2" value="ATTINY85V" x="11.5" y="14" smashed="yes" rot="R270">
+<element name="U1" library="Eigene-Rietig" library_urn="urn:adsk.eagle:library:40964436" package="SOIC8_200" package3d_urn="urn:adsk.eagle:package:41055619/3" value="ATTINY85V" x="11.5" y="14" smashed="yes" rot="R270">
 <attribute name="NAME" x="15" y="11.5" size="1" layer="25" font="vector" ratio="12" rot="R180" align="bottom-center"/>
 <attribute name="VALUE" x="22.5" y="11" size="1.27" layer="27" ratio="10"/>
 </element>
-<element name="SV1" library="con-lstb" library_urn="urn:adsk.eagle:library:162" package="MA03-1" package3d_urn="urn:adsk.eagle:package:8339/1" value="" x="3" y="11" smashed="yes" rot="R90">
+<element name="SV1" library="con-lstb" library_urn="urn:adsk.eagle:library:41989194" package="MA03-1" package3d_urn="urn:adsk.eagle:package:43315831/1" value="" x="3" y="11" smashed="yes" rot="R90">
 <attribute name="MF" value="" x="3" y="11" size="1.27" layer="27" rot="R90" display="off"/>
 <attribute name="MPN" value="" x="3" y="11" size="1.27" layer="27" rot="R90" display="off"/>
@@
 <attribute name="VALUE" x="10" y="25.5" size="1.27" layer="27" rot="R90"/>
 </element>
-<element name="Q2" library="SparkFun-DiscreteSemi" library_urn="urn:adsk.eagle:library:514" package="SOT23-3" package3d_urn="urn:adsk.eagle:package:38446/1" value="DMN3404L-7" x="12.5" y="23" smashed="yes" rot="R270">
+<element name="Q2" library="SparkFun-DiscreteSemi" library_urn="urn:adsk.eagle:library:514" package="SOT23-3" package3d_urn="urn:adsk.eagle:package:38446/2" value="5.8A/30V/35mΩ" x="12.5" y="23" smashed="yes" rot="R270">
 <attribute name="NAME" x="12.5" y="24.651" size="1" layer="25" font="vector" ratio="12" align="bottom-center"/>
 <attribute name="PROD_ID" value="TRANS-12988" x="14" y="23" size="1.27" layer="27" rot="R270" display="off"/>
 <attribute name="VALUE" x="12.5" y="27.5" size="0.6096" layer="27" font="vector" ratio="20" rot="R90" align="top-center"/>
-</element>
-<element name="J2" library="Eigene-Rietig" library_urn="urn:adsk.eagle:library:40964436" package="TAG-CONNECT_TC2030-MCP-NL" package3d_urn="urn:adsk.eagle:package:41146494/1" value="" x="1" y="-8.5" smashed="yes">
-<attribute name="NAME" x="0.365" y="-7.23" size="1.27" layer="25"/>
 </element>
 </elements>
@@
 <via x="12.5" y="21.5" extent="1-16" drill="0.3"/>
 <contactref element="Q2" pad="2"/>
-<contactref element="J2" pad="6"/>
-<wire x1="15" y1="21.5" x2="21" y2="25" width="0" layer="19" extent="1-1"/>
-<wire x1="12.5" y1="21.5" x2="15" y2="21.5" width="0" layer="19" extent="1-1"/>
-<wire x1="11.5" y1="22.05" x2="12.5" y2="21.5" width="0" layer="19" extent="1-1"/>
-<wire x1="11" y1="21" x2="11.5" y2="22.05" width="0" layer="19" extent="1-1"/>
-<wire x1="11.5" y1="20" x2="11" y2="21" width="0" layer="19" extent="1-1"/>
-<wire x1="9" y1="20" x2="11" y2="21" width="0" layer="19" extent="1-1"/>
-<wire x1="15.5" y1="18" x2="15" y2="21.5" width="0" layer="19" extent="1-1"/>
-<wire x1="16.65" y1="18" x2="15.5" y2="18" width="0" layer="19" extent="1-1"/>
-<wire x1="16.5" y1="14" x2="16.65" y2="18" width="0" layer="19" extent="1-1"/>
-<wire x1="18.5" y1="12.5" x2="16.5" y2="14" width="0" layer="19" extent="1-1"/>
-<wire x1="16" y1="11" x2="17.865" y2="11.81" width="0" layer="19" extent="1-1"/>
-<wire x1="13.5" y1="11" x2="16" y2="11" width="0" layer="19" extent="1-1"/>
-<wire x1="11.5" y1="10.5" x2="13.5" y2="11" width="0" layer="19" extent="1-1"/>
-<wire x1="10.65" y1="9.5" x2="11.5" y2="10.5" width="0" layer="19" extent="1-1"/>
-<wire x1="11.5" y1="8.5" x2="10.65" y2="9.5" width="0" layer="19" extent="1-1"/>
-<wire x1="10.65" y1="7.5" x2="11.5" y2="8.5" width="0" layer="19" extent="1-1"/>
-<wire x1="10" y1="6" x2="10.65" y2="7.5" width="0" layer="19" extent="1-1"/>
-<wire x1="10.5" y1="5" x2="10" y2="6" width="0" layer="19" extent="1-1"/>
-<wire x1="11.5" y1="6" x2="10.5" y2="5" width="0" layer="19" extent="1-1"/>
-<wire x1="11.5" y1="4" x2="10.5" y2="5" width="0" layer="19" extent="1-1"/>
-<wire x1="9" y1="5" x2="10" y2="6" width="0" layer="19" extent="1-1"/>
-<wire x1="7.85" y1="5" x2="9" y2="5" width="0" layer="19" extent="1-1"/>
-<wire x1="10.5" y1="12.5" x2="11.5" y2="10.5" width="0" layer="19" extent="1-1"/>
-<wire x1="8.346" y1="12.105" x2="10.5" y2="12.5" width="0" layer="19" extent="1-1"/>
-<wire x1="6.5" y1="12" x2="8.346" y2="12.105" width="0" layer="19" extent="1-1"/>
-<wire x1="3" y1="11" x2="6.5" y2="12" width="0" layer="19" extent="1-1"/>
-<wire x1="8.5" y1="25" x2="11.5" y2="22.05" width="0" layer="19" extent="1-1"/>
-<wire x1="6.5" y1="23.95" x2="8.5" y2="25" width="0" layer="19" extent="1-1"/>
-<wire x1="5" y1="24.5" x2="6.5" y2="23.95" width="0" layer="19" extent="1-1"/>
-<wire x1="3.5" y1="23.95" x2="5" y2="24.5" width="0" layer="19" extent="1-1"/>
-<wire x1="1" y1="25" x2="3.5" y2="23.95" width="0" layer="19" extent="1-1"/>
-<wire x1="16" y1="1.5" x2="11.5" y2="4" width="0" layer="19" extent="1-1"/>
-<wire x1="17.5" y1="1.65" x2="16" y2="1.5" width="0" layer="19" extent="1-1"/>
-<wire x1="19.5" y1="1.65" x2="17.5" y2="1.65" width="0" layer="19" extent="1-1"/>
-<wire x1="21" y1="1.5" x2="19.5" y2="1.65" width="0" layer="19" extent="1-1"/>
-<wire x1="1" y1="1" x2="7.85" y2="5" width="0" layer="19" extent="1-1"/>
-<wire x1="4.81" y1="-7.865" x2="1" y2="1" width="0" layer="19" extent="1-1"/>
 </signal>
 <signal name="N$1">
@@
 <wire x1="9.6" y1="23.95" x2="11.5" y2="23.95" width="0.3" layer="1"/>
 </signal>
-<signal name="MOSI">
-<contactref element="J2" pad="4"/>
-</signal>
-<signal name="!RESET">
-<contactref element="J2" pad="5"/>
-</signal>
-<signal name="SCK">
-<contactref element="J2" pad="3"/>
-</signal>
-<signal name="VCC">
-<contactref element="J2" pad="2"/>
-</signal>
-<signal name="MISO">
-<contactref element="J2" pad="1"/>
-</signal>
 </signals>
