File: EVmulator_T10_Compact.brd (EAGLE design)
At the start: 22 x 15 mm, 23 parts, among them IC1 ATTINY4/5/9/10, Q2 IRLML6244TRPBF

Commit message: * Modified Hardware
Parts:
- added R8: 100k, rcl:R0603
- added R9: 100R, rcl:R0603
- C2: value 10nF -> 100nF
- C3: value 1n8 -> 2n2
- D1: value 1N4007 -> B5819W-TP
- D3: value 15W - 15V TVS SD15-01FTG -> SD15-01FTG
- D4: value W8 - 4V7 -> BZX38450-C4V7X
- Q2: value IRLML6244TRPBF -> DMN3404L-7
- moved LED1 0.50 mm to (20.0, 7.50)
Connections:
- new net N$1: Q2.1, R9.1
- net CLK: now also R9.2; no longer Q2.1
- net RESET: now also R8.2
- net VCC: now also R8.1
Routing:
- net GND: track 1.15 -> 4.74 mm, vias 13 -> 20
- net VCC: track 18.8 -> 22.3 mm
- net N$1: track 0.00 -> 3.41 mm
- net DAT: track 11.1 -> 8.37 mm
- net RESET: track 6.45 -> 8.86 mm
- net CLK: track 6.15 -> 3.93 mm
- net CP: track 32.1 -> 32.7 mm
Other:
- board text added: "LED"
