File: EVmulator_T10_Compact.sch (EAGLE design)
At the start: 23 parts, among them IC1 ATTINY4/5/9/10, Q2 IRLML6244TRPBF

Commit message: * Modified Hardware
Parts:
- added R8: 100k, rcl:R-EU_R0603
- added R9: 100R, rcl:R-EU_R0603
- C2: value 10nF -> 100nF
- C3: value 1n8 -> 2n2
- D1: value 1N4007 -> B5819W-TP
- D3: value 15W - 15V TVS SD15-01FTG -> SD15-01FTG
- D4: value W8 - 4V7 -> BZX38450-C4V7X
- Q2: value IRLML6244TRPBF -> DMN3404L-7
Connections:
- new net N$1: Q2.G, R9.1
- net CLK: now also R9.2; no longer Q2.G
- net RESET: now also R8.2
- net VCC: now also R8.1
Other:
- moved on the sheet: D1, D3, Q2, R2, R3

Commit message: Updated readme and schematics
Other:
- note added: "LED: Reichelt 3034G3C-CSE-B"
Changed lines of the file:
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@@
 <text x="132.08" y="50.8" size="1.778" layer="91">6pin TagConnect
 Pinout 6pin ISP compatible</text>
+<text x="177.8" y="96.52" size="1.778" layer="91" rot="R180">LED: Reichelt 3034G3C-CSE-B</text>
 </plain>
 <instances>

Commit message: Annotated schematic a bit more, created new PDF of schematics
Other:
- note added: "Bypass reed switch for external switch"
- note added: "Close after programming (TPI does not like the LED)"
Changed lines of the file:
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@@
 Pinout 6pin ISP compatible</text>
 <text x="177.8" y="96.52" size="1.778" layer="91" rot="R180">LED: Reichelt 3034G3C-CSE-B</text>
+<text x="185.42" y="104.14" size="1.27" layer="91">Close after programming
+(TPI does not like the LED)</text>
+<text x="91.44" y="160.02" size="1.27" layer="91">Bypass reed switch for external switch</text>
 </plain>
 <instances>
